File: CASIO_RC-2/CASIO_RC-2.kicad_pcb (KiCad board)
At the start: 2 copper layers, 47 x 57 mm, 15 parts, among them J1 Conn_01x21_Pin, J2 Conn_01x02_Pin

Commit message: Updated PCB
Added all the little PCB details & fixed the hold spacing.
Other:
- outline, holes or cut-outs redrawn
- board text added: "+"
- board text added: "-"
Changed lines of the file:
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@@
 		(at 123.5 69)
 		(property "Reference" "J1"
-			(at 0 1.45 0)
+			(at 16.9 -9.7 0)
 			(unlocked yes)
 			(layer "F.SilkS")
@@
 		(at 131.55 91.5 -90)
 		(property "Reference" "J2"
-			(at 0 27.05 90)
+			(at 9.3 7.65 0)
 			(unlocked yes)
 			(layer "B.SilkS")
@@
 		(layer "B.SilkS")
 	)
+	(gr_circle
+		(center 129.2 100.4)
+		(end 129.9 101.1)
+		(stroke
+			(width 0.1)
+			(type default)
+		)
+		(fill no)
+		(layer "B.SilkS")
+	)
 	(gr_line
 		(start 102.3 81.9)
@@
 	)
 	(gr_circle
+		(center 101.310051 92.8)
+		(end 102.010051 93.5)
+		(stroke
+			(width 0.1)
+			(type default)
+		)
+		(fill no)
+		(layer "B.SilkS")
+	)
+	(gr_circle
 		(center 131 99)
 		(end 131.8 99.6)
@@
 		(layer "Edge.Cuts")
 	)
+	(gr_line
+		(start 129.8 101.7)
+		(end 130.1 102)
+		(stroke
+			(width 0.05)
+			(type default)
+		)
+		(layer "Edge.Cuts")
+	)
 	(gr_circle
 		(center 108.3 98.5)
@@
 		(layer "Edge.Cuts")
 	)
+	(gr_line
+		(start 138 102)
+		(end 138 99.5)
+		(stroke
+			(width 0.05)
+			(type default)
+		)
+		(layer "Edge.Cuts")
+	)
+	(gr_line
+		(start 147 102)
+		(end 147 45)
+		(stroke
+			(width 0.05)
+			(type default)
+		)
+		(layer "Edge.Cuts")
+	)
+	(gr_line
+		(start 103.9 101.7)
+		(end 129.8 101.7)
+		(stroke
+			(width 0.05)
+			(type default)
+		)
+		(layer "Edge.Cuts")
+	)
+	(gr_line
+		(start 103.9 101.7)
+		(end 103.7 102)
+		(stroke
+			(width 0.05)
+			(type default)
+		)
+		(layer "Edge.Cuts")
+	)
+	(gr_line
+		(start 139 102)
+		(end 139 99.5)
+		(stroke
+			(width 0.05)
+			(type default)
+		)
+		(layer "Edge.Cuts")
+	)
+	(gr_arc
+		(start 102.5 94.5)
+		(mid 103 95)
+		(end 102.5 95.5)
+		(stroke
+			(width 0.05)
+			(type default)
+		)
+		(layer "Edge.Cuts")
+	)
+	(gr_line
+		(start 100 45)
+		(end 100 94.5)
+		(stroke
+			(width 0.05)
+			(type default)
+		)
+		(layer "Edge.Cuts")
+	)
+	(gr_line
+		(start 100 102)
+		(end 103.7 102)
+		(stroke
+			(width 0.05)
+			(type default)
+		)
+		(layer "Edge.Cuts")
+	)
+	(gr_line
+		(start 147 45)
+		(end 100 45)
+		(stroke
+			(width 0.05)
+			(type default)
+		)
+		(layer "Edge.Cuts")
+	)
+	(gr_line
+		(start 100 94.5)
+		(end 102.5 94.5)
+		(stroke
+			(width 0.05)
+			(type default)
+		)
+		(layer "Edge.Cuts")
+	)
+	(gr_line
+		(start 138 102)
+		(end 130.1 102)
+		(stroke
+			(width 0.05)
+			(type default)
+		)
+		(layer "Edge.Cuts")
+	)
 	(gr_circle
 		(center 122 99)
@@
 		(layer "Edge.Cuts")
 	)
+	(gr_line
+		(start 139 102)
+		(end 147 102)
+		(stroke
+			(width 0.05)
+			(type default)
+		)
+		(layer "Edge.Cuts")
+	)
+	(gr_line
+		(start 100 95.5)
+		(end 100 102)
+		(stroke
+			(width 0.05)
+			(type default)
+		)
+		(layer "Edge.Cuts")
+	)
 	(gr_circle
 		(center 144.5 99.5)
@@
 		(layer "Edge.Cuts")
 	)
-	(gr_rect
-		(start 100 45)
-		(end 147 102)
+	(gr_arc
+		(start 138 99.5)
+		(mid 138.5 99)
+		(end 139 99.5)
+		(stroke
+			(width 0.05)
+			(type default)
+		)
+		(layer "Edge.Cuts")
+	)
+	(gr_line
+		(start 100 95.5)
+		(end 102.5 95.5)
 		(stroke
 			(width 0.05)
 			(type default)
 		)
-		(fill no)
 		(layer "Edge.Cuts")
 	)
@@
 		)
 	)
+	(gr_text "-"
+		(at 102.010051 93.3 0)
+		(layer "B.SilkS")
+		(effects
+			(font
+				(size 1 1)
+				(thickness 0.1)
+			)
+			(justify left bottom mirror)
+		)
+	)
+	(gr_text "+"
+		(at 129.9 100.9 0)
+		(layer "B.SilkS")
+		(effects
+			(font
+				(size 1 1)
+				(thickness 0.1)
+			)
+			(justify left bottom mirror)
+		)
+	)
